File: physical/isolator_input/isolator_input.sch (KiCad schematic (older format))
At the start: 20 parts, among them J1 Conn_01x04_Male, J2 Conn_01x03_Male, Q1 PN2222A, Q2 PN2222A, U1 H11L1, U2 H11L1

Commit message: opto-isolator board op-amp indicator
Parts:
- removed Q1, Q2: PN2222A, Package_TO_SOT_THT:TO-92_Inline, symbol Transistor_BJT:PN2222A
- removed R4, R8: 1k, Resistor_SMD:R_1206_3216Metric_Pad1.42x1.75mm_HandSolder, symbol Device:R
- added U3: MCP6002-xSN, Package_DIP:DIP-8_W7.62mm, symbol Amplifier_Operational:MCP6002-xSN
- C1, C2: symbol Device:CP1_Small -> Device:C
Connections:
- net +3V3: now also U3.8 (V+); no longer R3.2, R7.2
- net GNDA: now also R3.1, R7.1, U3.4 (V-)
- net Out01: now also U3.3 (+)
- net Out02: now also U3.5 (+)
- net at D2.1 (K): now also R3.2
- net at D2.2 (A): now also U3.1, U3.2 (-); no longer R3.1
- net at D4.1 (K): now also R7.2
- net at D4.2 (A): now also U3.6 (-), U3.7; no longer R7.1
Other:
- moved on the sheet: D1, D2, D3, D4, J1, J2, R1, R2, R3, R5, R6, R7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

Commit message: reverse polarity LED indicator
Connections:
- net +3V3: no longer C1.1, C2.1, R2.2, R6.2, U1.6, U2.6, U3.8 (V+)
- net GNDA: no longer R3.1, R7.1
- net at D2.1 (K): now also U3.1, U3.2 (-); no longer R3.2
- net at U3.6 (-), U3.7: now also D4.1 (K); no longer D4.2 (A)
- net VDD: now reaches R7.2
- net VDD: now also C1.1, C2.1, R2.2, R3.2, R6.2, U1.6, U2.6, U3.8 (V+); no longer D4.1 (K)
- new net: D2.2 (A), R3.1
- new net: D4.2 (A), R7.1
Other:
- moved on the sheet: D2, D4, R3, R7, U3C
Changed lines of the file:
@@
 L Device:LED D2
 U 1 1 5DD45999
-P 3950 2250
-F 0 "D2" V 4000 2450 50  0000 R CNN
-F 1 "LED" V 3900 2450 50  0000 R CNN
-F 2 "LED_SMD:LED_1206_3216Metric_Pad1.42x1.75mm_HandSolder" H 3950 2250 50  0001 C CNN
-F 3 "~" H 3950 2250 50  0001 C CNN
-	1    3950 2250
+P 4100 1950
+F 0 "D2" V 4150 1800 50  0000 R CNN
+F 1 "LED" V 4050 1850 50  0000 R CNN
+F 2 "LED_SMD:LED_1206_3216Metric_Pad1.42x1.75mm_HandSolder" H 4100 1950 50  0001 C CNN
+F 3 "~" H 4100 1950 50  0001 C CNN
+	1    4100 1950
 	0    -1   -1   0
 $EndComp
@@
 $EndComp
 $Comp
-L power:+3.3V #PWR0104
-U 1 1 5DD4C595
-P 2600 1450
-F 0 "#PWR0104" H 2600 1300 50  0001 C CNN
-F 1 "+3.3V" H 2615 1623 50  0000 C CNN
-F 2 "" H 2600 1450 50  0001 C CNN
-F 3 "" H 2600 1450 50  0001 C CNN
-	1    2600 1450
-	1    0    0    -1
-$EndComp
-$Comp
 L Device:R R3
 U 1 1 5DD52F20
-P 3950 2650
-F 0 "R3" V 4050 2700 50  0000 C CNN
-F 1 "330" V 4050 2550 50  0000 C CNN
-F 2 "Resistor_SMD:R_1206_3216Metric_Pad1.42x1.75mm_HandSolder" V 3880 2650 50  0001 C CNN
-F 3 "~" H 3950 2650 50  0001 C CNN
-	1    3950 2650
+P 4100 1550
+F 0 "R3" V 4200 1550 50  0000 C CNN
+F 1 "330" V 4000 1550 50  0000 C CNN
+F 2 "Resistor_SMD:R_1206_3216Metric_Pad1.42x1.75mm_HandSolder" V 4030 1550 50  0001 C CNN
+F 3 "~" H 4100 1550 50  0001 C CNN
+	1    4100 1550
 	-1   0    0    1
 $EndComp
@@
 Wire Wire Line
 	2600 1700 2600 1900
-$Comp
-L power:GNDA #PWR0101
-U 1 1 5DEB4084
-P 3950 2950
-F 0 "#PWR0101" H 3950 2700 50  0001 C CNN
-F 1 "GNDA" H 3955 2777 50  0000 C CNN
-F 2 "" H 3950 2950 50  0001 C CNN
-F 3 "" H 3950 2950 50  0001 C CNN
-	1    3950 2950
-	1    0    0    -1
-$EndComp
 Wire Wire Line
 	3000 2650 2900 2650
@@
 $EndComp
 $Comp
-L power:+3.3V #PWR0126
-U 1 1 5DEE9212
-P 2600 3550
-F 0 "#PWR0126" H 2600 3400 50  0001 C CNN
-F 1 "+3.3V" H 2615 3723 50  0000 C CNN
-F 2 "" H 2600 3550 50  0001 C CNN
-F 3 "" H 2600 3550 50  0001 C CNN
-	1    2600 3550
-	1    0    0    -1
-$EndComp
-$Comp
 L Device:R R7
 U 1 1 5DEE9218
-P 3950 4750
-F 0 "R7" V 3800 4950 50  0000 C CNN
-F 1 "330" V 3900 4950 50  0000 C CNN
-F 2 "Resistor_SMD:R_1206_3216Metric_Pad1.42x1.75mm_HandSolder" V 3880 4750 50  0001 C CNN
-F 3 "~" H 3950 4750 50  0001 C CNN
-	1    3950 4750
+P 4100 3750
+F 0 "R7" V 4200 3750 50  0000 C CNN
+F 1 "330" V 4000 3750 50  0000 C CNN
+F 2 "Resistor_SMD:R_1206_3216Metric_Pad1.42x1.75mm_HandSolder" V 4030 3750 50  0001 C CNN
+F 3 "~" H 4100 3750 50  0001 C CNN
+	1    4100 3750
 	-1   0    0    1
 $EndComp
@@
 L power:GNDA #PWR0127
 U 1 1 5DEE9234
-P 4500 3350
-F 0 "#PWR0127" H 4500 3100 50  0001 C CNN
-F 1 "GNDA" H 4505 3177 50  0000 C CNN
-F 2 "" H 4500 3350 50  0001 C CNN
-F 3 "" H 4500 3350 50  0001 C CNN
-	1    4500 3350
+P 4750 3250
+F 0 "#PWR0127" H 4750 3000 50  0001 C CNN
+F 1 "GNDA" H 4755 3077 50  0000 C CNN
+F 2 "" H 4750 3250 50  0001 C CNN
+F 3 "" H 4750 3250 50  0001 C CNN
+	1    4750 3250
 	1    0    0    -1
 $EndComp
@@
 Wire Wire Line
 	2600 1500 2600 1700
-Wire Wire Line
-	2600 1500 2600 1450
 Connection ~ 2600 1500
 Wire Wire Line
@@
 U 1 1 5DE56FD4
 P 3550 2100
-F 0 "U3" H 3550 1733 50  0000 C CNN
-F 1 "MCP6002-xSN" H 3550 1824 50  0000 C CNN
+F 0 "U3" H 3600 2250 50  0000 C CNN
+F 1 "MCP6002-xSN" H 3500 2350 50  0000 C CNN
 F 2 "Package_DIP:DIP-8_W7.62mm" H 3550 2100 50  0001 C CNN
 F 3 "http://ww1.microchip.com/downloads/en/DeviceDoc/21733j.pdf" H 3550 2100 50  0001 C CNN
@@
 U 2 1 5DE65914
 P 3550 4200
-F 0 "U3" H 3550 3833 50  0000 C CNN
-F 1 "MCP6002-xSN" H 3550 3924 50  0000 C CNN
+F 0 "U3" H 3550 4400 50  0000 C CNN
+F 1 "MCP6002-xSN" H 3500 4500 50  0000 C CNN
 F 2 "Package_DIP:DIP-8_W7.62mm" H 3550 4200 50  0001 C CNN
 F 3 "http://ww1.microchip.com/downloads/en/DeviceDoc/21733j.pdf" H 3550 4200 50  0001 C CNN
@@
 L Amplifier_Operational:MCP6002-xSN U3
 U 3 1 5DE66DDD
-P 4600 2950
-F 0 "U3" H 4558 2996 50  0000 L CNN
-F 1 "MCP6002-xSN" H 4558 2905 50  0000 L CNN
-F 2 "Package_DIP:DIP-8_W7.62mm" H 4600 2950 50  0001 C CNN
-F 3 "http://ww1.microchip.com/downloads/en/DeviceDoc/21733j.pdf" H 4600 2950 50  0001 C CNN
-	3    4600 2950
+P 4850 2850
+F 0 "U3" H 4808 2896 50  0000 L CNN
+F 1 "MCP6002-xSN" H 4808 2805 50  0000 L CNN
+F 2 "Package_DIP:DIP-8_W7.62mm" H 4850 2850 50  0001 C CNN
+F 3 "http://ww1.microchip.com/downloads/en/DeviceDoc/21733j.pdf" H 4850 2850 50  0001 C CNN
+	3    4850 2850
 	1    0    0    -1
 $EndComp
 Wire Wire Line
 	2900 2200 3250 2200
-Wire Wire Line
-	3950 2100 3850 2100
-Wire Wire Line
-	3250 1600 3950 1600
-Wire Wire Line
-	3250 1600 3250 2000
-Wire Wire Line
-	3950 1600 3950 2100
-Connection ~ 3950 2100
-Wire Wire Line
-	3950 2400 3950 2500
 $Comp
 L Device:LED D4
 U 1 1 5DEE91F4
-P 3950 4350
-F 0 "D4" V 4000 4550 50  0000 R CNN
-F 1 "LED" V 3900 4550 50  0000 R CNN
-F 2 "LED_SMD:LED_1206_3216Metric_Pad1.42x1.75mm_HandSolder" H 3950 4350 50  0001 C CNN
-F 3 "~" H 3950 4350 50  0001 C CNN
-	1    3950 4350
+P 4100 4050
+F 0 "D4" V 4150 3950 50  0000 R CNN
+F 1 "LED" V 4050 3950 50  0000 R CNN
+F 2 "LED_SMD:LED_1206_3216Metric_Pad1.42x1.75mm_HandSolder" H 4100 4050 50  0001 C CNN
+F 3 "~" H 4100 4050 50  0001 C CNN
+	1    4100 4050
 	0    -1   -1   0
 $EndComp
@@
 	2900 4300 3250 4300
 Wire Wire Line
-	3250 4100 3250 3700
-Wire Wire Line
-	3250 3700 3950 3700
-Wire Wire Line
-	3950 3700 3950 4200
-Wire Wire Line
-	3950 4200 3850 4200
-Connection ~ 3950 4200
-Wire Wire Line
-	3950 4500 3950 4600
-Wire Wire Line
-	3950 4900 3950 5050
-Wire Wire Line
-	3950 2800 3950 2950
-$Comp
-L power:+3.3V #PWR0112
-U 1 1 5DEF9091
-P 4500 2500
-F 0 "#PWR0112" H 4500 2350 50  0001 C CNN
-F 1 "+3.3V" H 4515 2673 50  0000 C CNN
-F 2 "" H 4500 2500 50  0001 C CNN
-F 3 "" H 4500 2500 50  0001 C CNN
-	1    4500 2500
-	1    0    0    -1
-$EndComp
-Wire Wire Line
-	4500 2500 4500 2650
-Wire Wire Line
-	4500 3250 4500 3350
-$Comp
-L power:GNDA #PWR0113
-U 1 1 5DF002FF
-P 3950 5050
-F 0 "#PWR0113" H 3950 4800 50  0001 C CNN
-F 1 "GNDA" H 3955 4877 50  0000 C CNN
-F 2 "" H 3950 5050 50  0001 C CNN
-F 3 "" H 3950 5050 50  0001 C CNN
-	1    3950 5050
-	1    0    0    -1
-$EndComp
+	4750 2400 4750 2550
+Wire Wire Line
+	4750 3150 4750 3250
+Wire Wire Line
+	2600 1400 2600 1500
+Connection ~ 3900 2100
+Wire Wire Line
+	3900 2100 3850 2100
+Wire Wire Line
+	4100 1700 4100 1800
+Wire Wire Line
+	3900 2100 4100 2100
+Wire Wire Line
+	3250 2000 3250 1850
+Wire Wire Line
+	3250 1850 3900 1850
+Wire Wire Line
+	3900 1850 3900 2100
+Wire Wire Line
+	3850 4200 3900 4200
+Wire Wire Line
+	3900 4200 3900 3950
+Wire Wire Line
+	3900 3950 3250 3950
+Wire Wire Line
+	3250 3950 3250 4100
+Connection ~ 3900 4200
+Wire Wire Line
+	3900 4200 4100 4200
+$Comp
+L power:VDD #PWR?
+U 1 1 5E018451
+P 4750 2400
+F 0 "#PWR?" H 4750 2250 50  0001 C CNN
+F 1 "VDD" H 4767 2573 50  0000 C CNN
+F 2 "" H 4750 2400 50  0001 C CNN
+F 3 "" H 4750 2400 50  0001 C CNN
+	1    4750 2400
+	1    0    0    -1
+$EndComp
+$Comp
+L power:VDD #PWR?
+U 1 1 5E01B6E5
+P 4100 3600
+F 0 "#PWR?" H 4100 3450 50  0001 C CNN
+F 1 "VDD" H 4117 3773 50  0000 C CNN
+F 2 "" H 4100 3600 50  0001 C CNN
+F 3 "" H 4100 3600 50  0001 C CNN
+	1    4100 3600
+	1    0    0    -1
+$EndComp
+$Comp
+L power:VDD #PWR?
+U 1 1 5E01BBA0
+P 2600 3550
+F 0 "#PWR?" H 2600 3400 50  0001 C CNN
+F 1 "VDD" H 2617 3723 50  0000 C CNN
+F 2 "" H 2600 3550 50  0001 C CNN
+F 3 "" H 2600 3550 50  0001 C CNN
+	1    2600 3550
+	1    0    0    -1
+$EndComp
+$Comp
+L power:VDD #PWR?
+U 1 1 5E01BFF8
+P 4100 1400
+F 0 "#PWR?" H 4100 1250 50  0001 C CNN
+F 1 "VDD" H 4117 1573 50  0000 C CNN
+F 2 "" H 4100 1400 50  0001 C CNN
+F 3 "" H 4100 1400 50  0001 C CNN
+	1    4100 1400
+	1    0    0    -1
+$EndComp
+$Comp
+L power:VDD #PWR?
+U 1 1 5E01C439
+P 2600 1400
+F 0 "#PWR?" H 2600 1250 50  0001 C CNN
+F 1 "VDD" H 2617 1573 50  0000 C CNN
+F 2 "" H 2600 1400 50  0001 C CNN
+F 3 "" H 2600 1400 50  0001 C CNN
+	1    2600 1400
+	1    0    0    -1
+$EndComp
